Commit message: 发现urdf转轴方向的问题，已经修复

File: legged_examples/legged_hunter/legged_hunter_description/urdf/hunter.urdf (robot description, URDF)
Before this commit: robot pai_12dof_v2_0312, 18 links, 17 joints
Joints:
- joint leg_l3_joint: axis 0 -1 0 -> 0 1 0
- joint leg_l5_joint: axis 0 -1 0 -> 0 1 0
